Commit message: finish

File: models/maze_bot.xacro (robot description, xacro)
@@ -49,5 +49,5 @@
       </visual>
       <collision>
-        <origin xyz="0 0 0" rpy="0 0 0" />
+        <origin xyz="0 0 0" rpy="1.570796 0 0" />
         <geometry>
           <cylinder length="0.04" radius="0.032"/>
